Commit message: Use GPIO tag in URDF.

File: ur_description/urdf/ur.ros2_control.xacro (robot description, xacro)
@@ -133,11 +133,11 @@
       </sensor>
       <!-- NOTE The following are joints used only for testing with fake hardware and will change in the future -->
-      <joint name="speed_scaling">
+      <gpio name="speed_scaling">
         <state_interface name="speed_scaling_factor"/>
         <param name="initial_speed_scaling_factor">1</param>
         <command_interface name="target_speed_fraction_cmd"/>
         <command_interface name="target_speed_fraction_async_success"/>
-      </joint>
-      <joint name="gpio">
+      </gpio>
+      <gpio name="gpio">
         <command_interface name="standard_digital_output_cmd_0"/>
         <command_interface name="standard_digital_output_cmd_1"/>
@@ -230,12 +230,12 @@
         <state_interface name="safety_status_bit_9"/>
         <state_interface name="safety_status_bit_10"/>
-      </joint>
-      <joint name="resend_robot_program">
+      </gpio>
+      <gpio name="resend_robot_program">
         <command_interface name="resend_robot_program_cmd"/>
         <command_interface name="resend_robot_program_async_success"/>
-      </joint>
-      <joint name="system_interface">
+      </gpio>
+      <gpio name="system_interface">
         <state_interface name="initialized"/>
-      </joint>
+      </gpio>
     </ros2_control>
   </xacro:macro>
